File: kicad/Xosera2/Xosera_HDMI.kicad_sch (KiCad schematic)
At the start: 30 parts, among them J10 sj, J4 5V, J5 3v3_5v_sel, J6 HDMI_A_1.4, J7 sj, J8 sj, J9 sj, U2 SII164

Commit message: Make a start on placement
Parts:
- C10, C11, C5, C6, C7, C8, C9: footprint pkl_dipol:C_0402 -> Capacitor_SMD:C_0402_1005Metric
- C14: footprint pkl_dipol:C_0603 -> Capacitor_SMD:C_0603_1608Metric
- C15, C16: footprint pkl_dipol:C_0603 -> Capacitor_SMD:C_0402_1005Metric
- J10: footprint pkl_jumpers:J_0603 -> Jumper:SolderJumper-2_P1.3mm_Open_RoundedPad1.0x1.5mm
- J5: footprint pkl_jumpers:J_NCNO_0903_30 -> Jumper:SolderJumper-3_P1.3mm_Bridged2Bar12_RoundedPad1.0x1.5mm
- J6: footprint pkl_connectors:HDMI-10029449-111RLF -> Connector_HDMI:HDMI_A_Amphenol_10029449-x01xLF_Horizontal
- J7, J8, J9: footprint pkl_jumpers:J_0903 -> Jumper:SolderJumper-3_P1.3mm_Open_RoundedPad1.0x1.5mm
- L1, L2, L3: footprint pkl_dipol:L_0402 -> Inductor_SMD:L_0603_1608Metric
- R1, R2, R3, R4, R5, R6, R7, R8, R9: footprint pkl_dipol:R_0402 -> Resistor_SMD:R_0603_1608Metric
- U2: footprint pkl_housings_qfp:TQFP-64-1EP_10x10mm_P0.5mm_EP5x5mm -> Package_QFP:TQFP-64_10x10mm_P0.5mm
Connections:
- net +3V3: now also J5.3; no longer J5.1
- net +5V: now also J5.1; no longer J5.3

Commit message: Replace all GALs with one 1504
Other:
- title: Xosera rosco_m68k daughterboard -> rosco_m68k Super Board
Changed lines of the file:
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@@
   (paper "A4")
   (title_block
-    (title "Xosera rosco_m68k daughterboard")
-    (date "2024-02-08")
+    (title "rosco_m68k Super Board")
+    (date "2024-02-11")
     (rev "0")
     (company "The Really Old-School Company Limited & XarkLabs")
     (comment 1 "Copyright (c)2023")
     (comment 2 "CERN OHL & MIT License")
+    (comment 3 "Featuring Xosera & MarkM's IDE")
   )
   (junction (at 257.81 118.11) (diameter 0) (color 0 0 0 0)

Commit message: Fix ERC (mostly) and sort out footprints etc
Parts:
- C10, C11, C5, C6, C7, C8, C9: symbol dvi-12bit-rescue:pkl_C_Small-pkl_device -> Device:C_Small
- C14, C15, C16: symbol dvi-12bit-rescue:pkl_C-pkl_device -> Device:C
- J10: symbol dvi-12bit-rescue:pkl_jumper-pkl_misc -> Jumper:Jumper_2_Open
- J5: symbol dvi-12bit-rescue:pkl_double_jumper_ncno-pkl_misc -> Jumper:Jumper_3_Bridged12
- J7, J8, J9: symbol dvi-12bit-rescue:pkl_double_jumper-pkl_misc -> Jumper:Jumper_3_Open
- L1, L2, L3: symbol dvi-12bit-rescue:pkl_L_Small-pkl_device -> Device:L_Small
- U2: footprint Package_QFP:TQFP-64_10x10mm_P0.5mm -> rosco_m68k:TQFP-64-1EP_10x10mm_P0.5mm_EP5x5mm; symbol dvi-12bit-rescue:SII164-pkl_lattice -> UPduino Imports:pkl_lattice_SII164
Connections:
- net +3V3: now also J7.3 (B), J8.3 (B), J9.3 (B), L1.2, L2.2, L3.2; no longer J7.1, J8.1, J9.1, L1.1, L2.1, L3.1
- net DKEN: now also J10.2 (B); no longer J10.1
- net GND: now also J10.1 (A), J7.1 (A), J8.1 (A), J9.1 (A); no longer J10.2, J7.3, J8.3, J9.3
- net PVCC: now also L2.1; no longer L2.2
- net TVDD: now also L3.1; no longer L3.2
- net VCC: now also L1.1; no longer L1.2
