File: kicad/Xosera2/Expansion_RAM.kicad_sch (KiCad schematic)
At the start: 16 parts, among them U2 AS6C8016, U3 AS6C8016, U4 AS6C8016, U5 AS6C8016

Commit message: Initial layout, delete some useless things
Connections:
- net A15: now also U2.18 (A18), U2.18 (A18), U2.18 (A18), U3.18 (A18), U4.18 (A18), U4.18 (A18), U4.18 (A18), U5.18 (A18); no longer U2.22 (A14), U2.22 (A14), U2.22 (A14), U3.22 (A14), U4.22 (A14), U4.22 (A14), U4.22 (A14), U5.22 (A14)
- net A16: now also U2.19 (A17), U2.19 (A17), U2.19 (A17), U3.19 (A17), U4.19 (A17), U4.19 (A17), U4.19 (A17), U5.19 (A17); no longer U2.21 (A15), U2.21 (A15), U2.21 (A15), U3.21 (A15), U4.21 (A15), U4.21 (A15), U4.21 (A15), U5.21 (A15)
- net A18: now also U2.21 (A15), U2.21 (A15), U2.21 (A15), U3.21 (A15), U4.21 (A15), U4.21 (A15), U4.21 (A15), U5.21 (A15); no longer U2.19 (A17), U2.19 (A17), U2.19 (A17), U3.19 (A17), U4.19 (A17), U4.19 (A17), U4.19 (A17), U5.19 (A17)
- net A19: now also U2.22 (A14), U2.22 (A14), U2.22 (A14), U3.22 (A14), U4.22 (A14), U4.22 (A14), U4.22 (A14), U5.22 (A14); no longer U2.18 (A18), U2.18 (A18), U2.18 (A18), U3.18 (A18), U4.18 (A18), U4.18 (A18), U4.18 (A18), U5.18 (A18)
- net A4: now also U2.1 (A4), U2.1 (A4), U2.1 (A4), U3.1 (A4), U4.1 (A4), U4.1 (A4), U4.1 (A4), U5.1 (A4); no longer U2.2 (A3), U2.2 (A3), U2.2 (A3), U3.2 (A3), U4.2 (A3), U4.2 (A3), U4.2 (A3), U5.2 (A3)
- net A5: now also U2.2 (A3), U2.2 (A3), U2.2 (A3), U3.2 (A3), U4.2 (A3), U4.2 (A3), U4.2 (A3), U5.2 (A3); no longer U2.1 (A4), U2.1 (A4), U2.1 (A4), U3.1 (A4), U4.1 (A4), U4.1 (A4), U4.1 (A4), U5.1 (A4)
- net D0: now also U2.10 (DQ3), U2.10 (DQ3), U2.10 (DQ3), U3.10 (DQ3), U4.10 (DQ3), U4.10 (DQ3), U4.10 (DQ3), U5.10 (DQ3); no longer U2.7 (DQ0), U2.7 (DQ0), U2.7 (DQ0), U3.7 (DQ0), U4.7 (DQ0), U4.7 (DQ0), U4.7 (DQ0), U5.7 (DQ0)
- net D1: now also U2.9 (DQ2), U2.9 (DQ2), U2.9 (DQ2), U3.9 (DQ2), U4.9 (DQ2), U4.9 (DQ2), U4.9 (DQ2), U5.9 (DQ2); no longer U2.8 (DQ1), U2.8 (DQ1), U2.8 (DQ1), U3.8 (DQ1), U4.8 (DQ1), U4.8 (DQ1), U4.8 (DQ1), U5.8 (DQ1)
- net D2: now also U2.8 (DQ1), U2.8 (DQ1), U2.8 (DQ1), U3.8 (DQ1), U4.8 (DQ1), U4.8 (DQ1), U4.8 (DQ1), U5.8 (DQ1); no longer U2.9 (DQ2), U2.9 (DQ2), U2.9 (DQ2), U3.9 (DQ2), U4.9 (DQ2), U4.9 (DQ2), U4.9 (DQ2), U5.9 (DQ2)
- net D3: now also U2.7 (DQ0), U2.7 (DQ0), U2.7 (DQ0), U3.7 (DQ0), U4.7 (DQ0), U4.7 (DQ0), U4.7 (DQ0), U5.7 (DQ0); no longer U2.10 (DQ3), U2.10 (DQ3), U2.10 (DQ3), U3.10 (DQ3), U4.10 (DQ3), U4.10 (DQ3), U4.10 (DQ3), U5.10 (DQ3)
- net D4: now also U2.16 (DQ7), U2.16 (DQ7), U2.16 (DQ7), U3.16 (DQ7), U4.16 (DQ7), U4.16 (DQ7), U4.16 (DQ7), U5.16 (DQ7); no longer U2.13 (DQ4), U2.13 (DQ4), U2.13 (DQ4), U3.13 (DQ4), U4.13 (DQ4), U4.13 (DQ4), U4.13 (DQ4), U5.13 (DQ4)
- net D5: now also U2.15 (DQ6), U2.15 (DQ6), U2.15 (DQ6), U3.15 (DQ6), U4.15 (DQ6), U4.15 (DQ6), U4.15 (DQ6), U5.15 (DQ6); no longer U2.14 (DQ5), U2.14 (DQ5), U2.14 (DQ5), U3.14 (DQ5), U4.14 (DQ5), U4.14 (DQ5), U4.14 (DQ5), U5.14 (DQ5)
- net D6: now also U2.14 (DQ5), U2.14 (DQ5), U2.14 (DQ5), U3.14 (DQ5), U4.14 (DQ5), U4.14 (DQ5), U4.14 (DQ5), U5.14 (DQ5); no longer U2.15 (DQ6), U2.15 (DQ6), U2.15 (DQ6), U3.15 (DQ6), U4.15 (DQ6), U4.15 (DQ6), U4.15 (DQ6), U5.15 (DQ6)
- net D7: now also U2.13 (DQ4), U2.13 (DQ4), U2.13 (DQ4), U3.13 (DQ4), U4.13 (DQ4), U4.13 (DQ4), U4.13 (DQ4), U5.13 (DQ4); no longer U2.16 (DQ7), U2.16 (DQ7), U2.16 (DQ7), U3.16 (DQ7), U4.16 (DQ7), U4.16 (DQ7), U4.16 (DQ7), U5.16 (DQ7)
- net VCC renamed +5VD
