File: kicad/Xosera2/IDE.kicad_sch (KiCad schematic)
At the start: 28 parts, among them J2 Conn_02x20_Odd_Even, J3 Conn_02x22_Odd_Even, Q1 2N2907, U3 74HCT241, U4 SN74HCT245DWR

Commit message: Fix ERC (mostly) and sort out footprints etc
Parts:
- J2: footprint Pin_Headers:Pin_Header_Straight_2x20_Pitch2.54mm -> Connector_IDC:IDC-Header_2x20_P2.54mm_Vertical
- J3: footprint Pin_Headers:Pin_Header_Straight_2x22_Pitch2.00mm -> Connector_PinHeader_2.00mm:PinHeader_2x22_P2.00mm_Vertical
- JP1: footprint Pin_Headers:Pin_Header_Straight_1x02_Pitch2.54mm -> Connector_PinHeader_2.54mm:PinHeader_1x02_P2.54mm_Vertical; symbol ata-ide-rescue:Jumper-Device -> Jumper:Jumper_2_Open
- TP1, TP2, TP3: footprint Measurement_Points:Measurement_Point_Round-TH_Big -> TestPoint:TestPoint_Pad_D1.0mm
- U3: symbol ata-ide-rescue:74LS241-74xx_IEEE -> 74xx_IEEE:74LS241
Connections:
- net +5V: no longer C1.1, C1.1, C1.1, C1.1, C1.1, C1.1, C7.1, C8.1, C9.1, JP1.1, Q1.1 (E), R1.1, R2.1, TP1.1, U3.20 (VCC), U3.20 (VCC), U4.20 (VCC), U4.20 (VCC)
- new net +5VD: C1.1, C1.1, C1.1, C1.1, C1.1, C1.1, C7.1, C8.1, C9.1, JP1.1 (A), Q1.1 (E), R1.1, R2.1, TP1.1, U3.20 (VCC), U3.20 (VCC), U4.20 (VCC), U4.20 (VCC)
Other:
- note removed: "NOTE: This ATF750 may be replaced with an 22V10 if less complex logic is required,e.g. if simpler ~{RD} and ~{DTACK} logic is required."
- moved on the sheet: JP3, JP4, JP5

Commit message: Initial layout, delete some useless things
Parts:
- removed C8: 10u, Capacitor_SMD:CP_Elec_6.3x5.4, symbol Device:C_Polarized
- removed TP2, TP3: TestPoint, TestPoint:TestPoint_Pad_D1.0mm, symbol Connector:TestPoint
Connections:
- net ~{IRQ3}: now also JP5.2 (B); no longer JP3.2 (B)
- net ~{IRQ6}: now also JP3.2 (B); no longer JP5.2 (B)
- net at JP5.1 (A): now also U3.9 (O0); no longer U3.5 (O2)
- net at JP3.1 (A): now also U3.5 (O2); no longer U3.9 (O0)
Other:
- moved on the sheet: JP3, JP5
Changed lines of the file:
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@@
   (junction (at 59.69 160.02) (diameter 0) (color 0 0 0 0)
   )
-  (junction (at 90.17 160.02) (diameter 0) (color 0 0 0 0)
-  )
   (junction (at 203.2 120.65) (diameter 0) (color 0 0 0 0)
   )
@@
   )
   (junction (at 80.01 160.02) (diameter 0) (color 0 0 0 0)
-  )
-  (junction (at 90.17 172.72) (diameter 0) (color 0 0 0 0)
   )
   (junction (at 274.32 125.73) (diameter 0) (color 0 0 0 0)
@@
     (stroke (width 0) (type default))
   )
-  (wire (pts (xy 80.01 172.72) (xy 90.17 172.72))
+  (wire (pts (xy 80.01 172.72) (xy 100.33 172.72))
     (stroke (width 0) (type default))
   )
@@
     (stroke (width 0) (type default))
   )
-  (wire (pts (xy 90.17 160.02) (xy 90.17 162.56))
-    (stroke (width 0) (type default))
-  )
   (wire (pts (xy 86.36 107.95) (xy 93.98 107.95))
     (stroke (width 0) (type default))
@@
     (stroke (width 0) (type default))
   )
-  (wire (pts (xy 100.33 172.72) (xy 90.17 172.72))
-    (stroke (width 0) (type default))
-  )
   (wire (pts (xy 19.05 160.02) (xy 19.05 162.56))
     (stroke (width 0) (type default))
@@
     (stroke (width 0) (type default))
   )
-  (wire (pts (xy 90.17 172.72) (xy 90.17 170.18))
-    (stroke (width 0) (type default))
-  )
   (wire (pts (xy 248.92 143.51) (xy 232.41 143.51))
     (stroke (width 0) (type default))
@@
     (stroke (width 0) (type default))
   )
-  (wire (pts (xy 90.17 160.02) (xy 100.33 160.02))
-    (stroke (width 0) (type default))
-  )
   (wire (pts (xy 132.08 105.41) (xy 140.97 105.41))
     (stroke (width 0) (type default))
@@
     (stroke (width 0) (type default))
   )
-  (wire (pts (xy 80.01 160.02) (xy 90.17 160.02))
+  (wire (pts (xy 80.01 160.02) (xy 100.33 160.02))
     (stroke (width 0) (type default))
   )
@@
     )
   )
-  (symbol (lib_id "Jumper:SolderJumper_2_Bridged") (at 123.19 60.96 0) (unit 1)
-    (in_bom yes) (on_board yes) (dnp no)
-    (property "Reference" "JP5" (at 123.19 55.753 0)
-      (effects (font (size 1.27 1.27)))
-    )
-    (property "Value" "SolderJumper_2_Bridged" (at 129.54 58.42 0)
-      (effects (font (size 1.27 1.27)))
-    )
-    (property "Footprint" "Jumper:SolderJumper-2_P1.3mm_Bridged_RoundedPad1.0x1.5mm" (at 123.19 60.96 0)
-      (effects (font (size 1.27 1.27)) hide)
-    )
-    (property "Datasheet" "~" (at 123.19 60.96 0)
+  (symbol (lib_id "Jumper:SolderJumper_2_Bridged") (at 123.19 38.1 0) (unit 1)
+    (in_bom yes) (on_board yes) (dnp no)
+    (property "Reference" "JP5" (at 123.19 32.893 0)
+      (effects (font (size 1.27 1.27)))
+    )
+    (property "Value" "SolderJumper_2_Bridged" (at 129.54 35.56 0)
+      (effects (font (size 1.27 1.27)))
+    )
+    (property "Footprint" "Jumper:SolderJumper-2_P1.3mm_Bridged_RoundedPad1.0x1.5mm" (at 123.19 38.1 0)
+      (effects (font (size 1.27 1.27)) hide)
+    )
+    (property "Datasheet" "~" (at 123.19 38.1 0)
       (effects (font (size 1.27 1.27)) hide)
     )
@@
     )
   )
-  (symbol (lib_id "Connector:TestPoint") (at 39.37 172.72 180) (unit 1)
-    (in_bom yes) (on_board yes) (dnp no)
-    (property "Reference" "TP3" (at 40.64 176.53 0)
-      (effects (font (size 1.27 1.27)) (justify right))
-    )
-    (property "Value" "TestPoint" (at 35.56 179.07 0)
-      (effects (font (size 1.27 1.27)) (justify right))
-    )
-    (property "Footprint" "TestPoint:TestPoint_Pad_D1.0mm" (at 34.29 172.72 0)
-      (effects (font (size 1.27 1.27)) hide)
-    )
-    (property "Datasheet" "~" (at 34.29 172.72 0)
-      (effects (font (size 1.27 1.27)) hide)
-    )
-    (pin "1")
-    (instances
-      (project "ata-ide"
-        (path "/271ea45f-b126-4d8c-90a7-5005445be9f6"
-          (reference "TP3") (unit 1)
-        )
-      )
-      (project "Xosera2"
-        (path "/e3ab5ddd-7cd3-46c7-91c9-5fc78e7ae4ac/4ee056bd-bf09-4e04-a133-a9171db1e0fc"
-          (reference "TP24") (unit 1)
-        )
-      )
-    )
-  )
   (symbol (lib_id "Device:R") (at 130.81 173.99 180) (unit 1)
     (in_bom yes) (on_board yes) (dnp no)
@@
         (path "/e3ab5ddd-7cd3-46c7-91c9-5fc78e7ae4ac/4ee056bd-bf09-4e04-a133-a9171db1e0fc"
           (reference "#PWR0138") (unit 1)
-        )
-      )
-    )
-  )
-  (symbol (lib_id "Device:C_Polarized") (at 90.17 166.37 0) (unit 1)
-    (in_bom yes) (on_board yes) (dnp no)
-    (property "Reference" "C8" (at 93.1672 165.2016 0)
-      (effects (font (size 1.27 1.27)) (justify left))
-    )
-    (property "Value" "10u" (at 93.1672 167.513 0)
-      (effects (font (size 1.27 1.27)) (justify left))
-    )
-    (property "Footprint" "Capacitor_SMD:CP_Elec_6.3x5.4" (at 91.1352 170.18 0)
-      (effects (font (size 1.27 1.27)) hide)
-    )
-    (property "Datasheet" "~" (at 90.17 166.37 0)
-      (effects (font (size 1.27 1.27)) hide)
-    )
-    (property "LCSC" "C4747963" (at 90.17 166.37 0)
-      (effects (font (size 1.27 1.27)) hide)
-    )
-    (pin "1")
-    (pin "2")
-    (instances
-      (project "ata-ide"
-        (path "/271ea45f-b126-4d8c-90a7-5005445be9f6"
-          (reference "C8") (unit 1)
-        )
-      )
-      (project "Xosera2"
-        (path "/e3ab5ddd-7cd3-46c7-91c9-5fc78e7ae4ac/4ee056bd-bf09-4e04-a133-a9171db1e0fc"
-          (reference "C74") (unit 1)
         )
       )
@@
     )
   )
-  (symbol (lib_id "Jumper:SolderJumper_2_Open") (at 123.19 38.1 0) (unit 1)
-    (in_bom yes) (on_board yes) (dnp no)
-    (property "Reference" "JP3" (at 123.19 32.893 0)
-      (effects (font (size 1.27 1.27)))
-    )
-    (property "Value" "SolderJumper_2_Open" (at 129.54 35.56 0)
-      (effects (font (size 1.27 1.27)))
-    )
-    (property "Footprint" "Jumper:SolderJumper-2_P1.3mm_Open_RoundedPad1.0x1.5mm" (at 123.19 38.1 0)
-      (effects (font (size 1.27 1.27)) hide)
-    )
-    (property "Datasheet" "~" (at 123.19 38.1 0)
+  (symbol (lib_id "Jumper:SolderJumper_2_Open") (at 123.19 60.96 0) (unit 1)
+    (in_bom yes) (on_board yes) (dnp no)
+    (property "Reference" "JP3" (at 123.19 55.753 0)
+      (effects (font (size 1.27 1.27)))
+    )
+    (property "Value" "SolderJumper_2_Open" (at 129.54 58.42 0)
+      (effects (font (size 1.27 1.27)))
+    )
+    (property "Footprint" "Jumper:SolderJumper-2_P1.3mm_Open_RoundedPad1.0x1.5mm" (at 123.19 60.96 0)
+      (effects (font (size 1.27 1.27)) hide)
+    )
+    (property "Datasheet" "~" (at 123.19 60.96 0)
       (effects (font (size 1.27 1.27)) hide)
     )
@@
         )
       )
-    )
-  )
-  (symbol (lib_id "Connector:TestPoint") (at 29.21 172.72 180) (unit 1)
-    (in_bom yes) (on_board yes) (dnp no)
-    (property "Reference" "TP2" (at 30.48 176.53 0)
-      (effects (font (size 1.27 1.27)) (justify right))
-    )
-    (property "Value" "TestPoint" (at 25.4 179.07 0)
-      (effects (font (size 1.27 1.27)) (justify right))
-    )
-    (property "Footprint" "TestPoint:TestPoint_Pad_D1.0mm" (at 24.13 172.72 0)
-      (effects (font (size 1.27 1.27)) hide)
-    )
-    (property "Datasheet" "~" (at 24.13 172.72 0)
-      (effects (font (size 1.27 1.27)) hide)
-    )
-    (pin "1")
-    (instances
-      (project "ata-ide"
-        (path "/271ea45f-b126-4d8c-90a7-5005445be9f6"
-          (reference "TP2") (unit 1)
-        )
-      )
-      (project "Xosera2"
-        (path "/e3ab5ddd-7cd3-46c7-91c9-5fc78e7ae4ac/4ee056bd-bf09-4e04-a133-a9171db1e0fc"
-          (reference "TP23") (unit 1)
-        )
-      )
