File: kicad/Xosera2/Xosera2.kicad_pcb (KiCad board)
At the start: 2 copper layers, 160 x 100 mm, 158 parts, among them IC1 93LC56BT-I/OT, IC10 SN74AUP2G125DCUR, IC11 TXB0108DQSR, IC12 TXB0108DQSR, IC2 ICE40UP5K-SG48ITR, IC3 FT232H, IC4 AP2127K-3.3, IC5 AP2127K-1.2, IC6 SII164, IC7 GAL22V10, IC8 74HCT74, IC9 ATF16V8BQL, J1 Conn_02x32_Odd_Even, J10 Conn_01x06_Male, J2 5V, J3 sj, J4 sj, J5 sj, J6 sj, J7 3v3_5v_sel, J8 HDMI_A_1.4, J9 47589-0001, Q1 SG-210STF 12.0000ML3, Q2 2N3904, U1 W25Q32JVSSIM

Commit message: Fix ERC (mostly) and sort out footprints etc
Parts:
- added C59: 100n, Capacitor_SMD:C_0402_1005Metric, F.Cu at (-221.2, 98.8)
- added C60: 100n, Capacitor_SMD:C_0402_1005Metric, F.Cu at (-221.2, 100.8)
- added C61: 100n, Capacitor_SMD:C_0402_1005Metric, F.Cu at (-221.2, 102.8)
- added C62: 100n, Capacitor_SMD:C_0402_1005Metric, F.Cu at (-221.2, 104.7)
- added C67: 100n, Capacitor_SMD:C_0402_1005Metric, F.Cu at (502.8, 77.7)
- added C68: 100n, Capacitor_SMD:C_0402_1005Metric, F.Cu at (502.8, 79.7)
- added C69: 100n, Capacitor_SMD:C_0402_1005Metric, F.Cu at (502.8, 81.6)
- added C70: 100n, Capacitor_SMD:C_0402_1005Metric, F.Cu at (502.8, 83.6)
- added C71: 100n, Capacitor_SMD:C_0402_1005Metric, F.Cu at (502.8, 85.6)
- added C72: 100n, Capacitor_SMD:C_0402_1005Metric, F.Cu at (502.8, 87.5)
- added C73: 100u, Capacitor_SMD:CP_Elec_6.3x5.4, F.Cu at (506.6, 64.5)
- added C74: 10u, Capacitor_SMD:CP_Elec_6.3x5.4, F.Cu at (506.6, 72.6)
- added C75: 4u7, Capacitor_SMD:C_0603_1608Metric, F.Cu at (518.3, 61.7)
- added D3: LED, LED_SMD:LED_0603_1608Metric, F.Cu at (518.8, 78.0)
- added IC13: 74HCT241, Package_SO:SOIC-20W_7.5x12.8mm_P1.27mm, F.Cu at (501.7, 53.2)
- added IC14: SN74HCT245DWR, Package_SO:SOIC-20W_7.5x12.8mm_P1.27mm, F.Cu at (514.6, 53.2)
- added J11: Conn_02x05_Odd_Even, Connector_IDC:IDC-Header_2x05_P2.54mm_Vertical, F.Cu at (239.6, 255.6)
- added J12: Conn_02x20_Odd_Even, Connector_IDC:IDC-Header_2x20_P2.54mm_Vertical, F.Cu at (488.5, 52.2)
- added J13: Conn_02x22_Odd_Even, Connector_PinHeader_2.00mm:PinHeader_2x22_P2.00mm_Vertical, F.Cu at (497.3, 62.4)
- added J14: Conn_02x07_Odd_Even, Connector_IDC:IDC-Header_2x07_P2.54mm_Vertical, F.Cu at (227.6, 255.6)
- added J15: Conn_02x05_Odd_Even, Connector_IDC:IDC-Header_2x05_P2.54mm_Vertical, F.Cu at (251.5, 255.6)
- added JP3: Pin 20 5V Supply, Connector_PinHeader_2.54mm:PinHeader_1x02_P2.54mm_Vertical, F.Cu at (506.5, 79.0)
- added JP4: SolderJumper_2_Bridged, Jumper:SolderJumper-2_P1.3mm_Bridged_Pad1.0x1.5mm, F.Cu at (514.1, 62.2)
- added JP5: SolderJumper_2_Open, Jumper:SolderJumper-2_P1.3mm_Open_RoundedPad1.0x1.5mm, F.Cu at (514.1, 65.7)
- added JP6: SolderJumper_2_Open, Jumper:SolderJumper-2_P1.3mm_Open_RoundedPad1.0x1.5mm, F.Cu at (514.1, 69.3)
- added JP7: SolderJumper_2_Bridged, Jumper:SolderJumper-2_P1.3mm_Bridged_RoundedPad1.0x1.5mm, F.Cu at (514.1, 72.8)
- added Q3: 2N2907, Package_TO_SOT_SMD:SOT-23, F.Cu at (514.3, 78.9)
- added R26: 330, Resistor_SMD:R_0603_1608Metric, F.Cu at (518.3, 64.2)
- added R27: 10k, Resistor_SMD:R_0603_1608Metric, F.Cu at (518.3, 66.7)
- added R28: 4k7, Resistor_SMD:R_0603_1608Metric, F.Cu at (518.3, 69.2)
- added R29: 10k, Resistor_SMD:R_0603_1608Metric, F.Cu at (518.3, 71.7)
- added R30: 10K, Resistor_SMD:R_0603_1608Metric, F.Cu at (236.3, 273.1)
- added R31: 10K, Resistor_SMD:R_0603_1608Metric, F.Cu at (236.3, 275.6)
- added R32: 10K, Resistor_SMD:R_0603_1608Metric, F.Cu at (236.3, 278.1)
- added R33: 10K, Resistor_SMD:R_0603_1608Metric, F.Cu at (236.3, 280.6)
- added TP22: TestPoint, TestPoint:TestPoint_Pad_D1.0mm, F.Cu at (510.4, 78.2)
- added TP23: TestPoint, TestPoint:TestPoint_Pad_D1.0mm, F.Cu at (510.4, 81.3)
- added TP24: TestPoint, TestPoint:TestPoint_Pad_D1.0mm, F.Cu at (510.4, 84.3)
- added U2: AS6C8016, Package_SO:TSOP-II-44_10.16x18.41mm_P0.8mm, F.Cu at (-215.5, 87.8)
- added U3: AS6C8016, Package_SO:TSOP-II-44_10.16x18.41mm_P0.8mm, F.Cu at (-201.3, 87.8)
- added U4: AS6C8016, Package_SO:TSOP-II-44_10.16x18.41mm_P0.8mm, F.Cu at (-187.0, 87.8)
- added U5: AS6C8016, Package_SO:TSOP-II-44_10.16x18.41mm_P0.8mm, F.Cu at (-172.8, 87.8)
- added U6: AS6C8016, Package_SO:TSOP-II-44_10.16x18.41mm_P0.8mm, F.Cu at (-158.5, 87.8)
- added U7: AS6C8016, Package_SO:TSOP-II-44_10.16x18.41mm_P0.8mm, F.Cu at (-144.3, 87.8)
- added U8: AS6C8016, Package_SO:TSOP-II-44_10.16x18.41mm_P0.8mm, F.Cu at (-130.0, 87.8)
- added U9: AS6C8016, Package_SO:TSOP-II-44_10.16x18.41mm_P0.8mm, F.Cu at (-115.8, 87.8)
- C1, C11, C12, C13, C14, C15, C16, C2, C22, C26, C28, C3, C31, C4, C6, C7, C9: value 0.1u -> 100n; footprint Capacitor_SMD:C_0603_1608Metric -> Capacitor_SMD:C_0402_1005Metric
- C20: value 0.1u -> 100m; footprint Capacitor_SMD:C_0603_1608Metric -> Capacitor_SMD:C_0402_1005Metric
- C44, C45, C48, C50, C51, C52, C54, C56, C58: value 100nF -> 100n; footprint Capacitor_SMD:C_0603_1608Metric -> Capacitor_SMD:C_0402_1005Metric
- C46: value 100uF -> 100u; footprint Capacitor_THT:CP_Radial_D5.0mm_P2.50mm -> Capacitor_SMD:CP_Elec_6.3x5.4
- C47: value 220uF -> 220u; footprint Capacitor_THT:CP_Radial_D6.3mm_P2.50mm -> Capacitor_SMD:CP_Elec_6.3x5.4
- C49, C53, C55, C57: value 100nF -> 100n; footprint Capacitor_SMD:C_0805_2012Metric -> Capacitor_SMD:C_0402_1005Metric
- IC6: footprint Package_QFP:TQFP-64_10x10mm_P0.5mm -> rosco_m68k:TQFP-64-1EP_10x10mm_P0.5mm_EP5x5mm
- IC7: value GAL22V10 -> ATF1504AS-TQFP100; footprint Package_DIP:DIP-24_W7.62mm_LongPads -> Package_QFP:TQFP-100_14x14mm_P0.5mm
- IC9: value ATF16V8BQL -> SN74HCT245DWR; footprint Package_DIP:DIP-20_W7.62mm_Socket_LongPads -> Package_SO:SOIC-20W_7.5x12.8mm_P1.27mm
- moved C49 539.1 mm to (-152.0, 104.8)
- moved C53 539.1 mm to (-139.0, 104.5)
- moved C48 464.4 mm to (-177.5, 107.6)
- moved C54 464.4 mm to (-178.2, 101.5)
- moved IC9 296.1 mm to (514.7, 98.0)
Connections:
- net /Xosera_Bus/~{BUS_RESET} renamed /Xosera_Bus/~{3V3_RESET}
- net IPL1 renamed /Xosera_Bus/~{IRQ2}
- C48 pad 1: +5V -> +3.3V
- C49 pad 1: +3V3 -> +3.3V
- C53 pad 1: +5VD -> +3.3V
- C54 pad 1: +5V -> +3.3V
- C56 pad 1: +5V -> +5VD
- C57 pad 1: +5VD -> +3V3
- C58 pad 1: +5V -> +5VD
- H1 pad 1: (no net) -> GND
- H2 pad 1: (no net) -> GND
- H3 pad 1: (no net) -> GND
- H4 pad 1: (no net) -> GND
- IC11 pad 1: BUS_DATA0 -> /Xosera_Bus/3V3_D8
- IC11 pad 10: BUS_DATA7 -> /Xosera_Bus/3V3_D15
- IC11 pad 11: 68_D15 -> /Xosera_Bus/5V_D15
- IC11 pad 12: 68_D14 -> /Xosera_Bus/5V_D14
- IC11 pad 13: 68_D13 -> /Xosera_Bus/5V_D13
- IC11 pad 14: 68_D12 -> /Xosera_Bus/5V_D12
- IC11 pad 17: 68_D11 -> /Xosera_Bus/5V_D11
- IC11 pad 18: 68_D10 -> /Xosera_Bus/5V_D10
- IC11 pad 19: 68_D9 -> /Xosera_Bus/5V_D9
- IC11 pad 2: BUS_DATA1 -> /Xosera_Bus/3V3_D9
- IC11 pad 20: 68_D8 -> /Xosera_Bus/5V_D8
- IC11 pad 3: BUS_DATA2 -> /Xosera_Bus/3V3_D10
- IC11 pad 4: BUS_DATA3 -> /Xosera_Bus/3V3_D11
- IC11 pad 6: FPGA_CS -> /Xosera_Bus/~{FPGA_CS}
- IC11 pad 7: BUS_DATA4 -> /Xosera_Bus/3V3_D12
- IC11 pad 8: BUS_DATA5 -> /Xosera_Bus/3V3_D13
- IC11 pad 9: BUS_DATA6 -> /Xosera_Bus/3V3_D14
- IC12 pad 1: BUS_BYTESEL -> /Xosera_Bus/3V3_BYTESEL
- IC12 pad 10: ~{JBUS_RESET} -> /Xosera_Bus/~{J3V3_RESET}
- IC12 pad 11: RESET -> /Xosera_Bus/~{RESET}
- IC12 pad 12: RnW -> /Xosera_Bus/R~{W}
- IC12 pad 13: FPGA_CS -> /Xosera_Bus/~{FPGA_CS}
- IC12 pad 14: A7 -> /Xosera_Bus/A7
- IC12 pad 17: A4 -> /Xosera_Bus/A4
- IC12 pad 18: A3 -> /Xosera_Bus/A3
- IC12 pad 19: A2 -> /Xosera_Bus/A2
- IC12 pad 2: BUS_REG_NUM0 -> /Xosera_Bus/3V3_REG_NUM0
- IC12 pad 20: A1 -> /Xosera_Bus/A1
- IC12 pad 3: BUS_REG_NUM1 -> /Xosera_Bus/3V3_REG_NUM1
- IC12 pad 4: BUS_REG_NUM2 -> /Xosera_Bus/3V3_REG_NUM2
- IC12 pad 7: BUS_REG_NUM3 -> /Xosera_Bus/3V3_REG_NUM3
- IC12 pad 8: /Xosera_Bus/~{BUS_CS} -> /Xosera_Bus/~{3V3_XOSERA_CS}
- IC12 pad 9: /Xosera_Bus/BUS_R~{W} -> /Xosera_Bus/3V3_R~{W}
- IC2 pad 10: /Xosera_Bus/UD_IRQ -> /Xosera_Bus/XOSERA_IRQ
- IC2 pad 23: BUS_REG_NUM0 -> /Xosera_Bus/3V3_REG_NUM0
- IC2 pad 25: BUS_REG_NUM1 -> /Xosera_Bus/3V3_REG_NUM1
- IC2 pad 26: BUS_REG_NUM2 -> /Xosera_Bus/3V3_REG_NUM2
- IC2 pad 27: BUS_REG_NUM3 -> /Xosera_Bus/3V3_REG_NUM3
- IC2 pad 28: BUS_DATA7 -> /Xosera_Bus/3V3_D15
- IC2 pad 31: BUS_DATA0 -> /Xosera_Bus/3V3_D8
- IC2 pad 34: BUS_DATA2 -> /Xosera_Bus/3V3_D10
- IC2 pad 36: BUS_DATA4 -> /Xosera_Bus/3V3_D12
- IC2 pad 37: BUS_DATA1 -> /Xosera_Bus/3V3_D9
- IC2 pad 38: BUS_DATA6 -> /Xosera_Bus/3V3_D14
- IC2 pad 39: /Xosera_Bus/BUS_R~{W} -> /Xosera_Bus/3V3_R~{W}
- IC2 pad 40: BUS_BYTESEL -> /Xosera_Bus/3V3_BYTESEL
- IC2 pad 41: /Xosera_Bus/~{BUS_CS} -> /Xosera_Bus/~{3V3_XOSERA_CS}
- IC2 pad 42: BUS_DATA5 -> /Xosera_Bus/3V3_D13
- IC2 pad 43: BUS_DATA3 -> /Xosera_Bus/3V3_D11
- IC7 pad 1: SEL_1 -> unconnected-(IC7-GCLR/I-Pad1)
- IC7 pad 10: RnW -> /Xosera_Bus/~{FPGA_CS}
- IC7 pad 11: /Xosera_Bus/UD_IRQ -> /IDE/~{LSEL}
- IC7 pad 12: GND -> /IDE/~{CS3}
- IC7 pad 13: unconnected-(IC7-I13-Pad13) -> +5V
- IC7 pad 14: unconnected-(IC7-IO1-Pad14) -> /Xosera_Bus/GLUE_TDI
- IC7 pad 15: IRQRS -> /IDE/~{USEL}
- IC7 pad 16: FPGA_CS -> /IDE/~{CS1}
- IC7 pad 17: unconnected-(IC7-I04-Pad17) -> /Expansion_RAM/W~{R}
- IC7 pad 18: FPGA_R -> unconnected-(IC7-I/O-Pad18)
- IC7 pad 19: OIRQ -> GND
- IC7 pad 2: FC0 -> /Xosera_Bus/XOSERA_IRQ
- IC7 pad 20: FPGA_W -> /Xosera_Bus/RAM_EN_2
- IC7 pad 21: unconnected-(IC7-IO8-Pad21) -> /Xosera_Bus/RAM_EN_1
- IC7 pad 22: VPA -> /Xosera_Bus/A2
- IC7 pad 23: DTACK -> /Xosera_Bus/GLUE_TMS
- IC7 pad 24: +5V -> /Xosera_Bus/IRQRS
- IC7 pad 3: FC1 -> +5V
- IC7 pad 4: FC2 -> /Xosera_Bus/~{IDE_CS}
- IC7 pad 5: AS -> /Xosera_Bus/~{UDS}
- IC7 pad 6: A1 -> /Xosera_Bus/R~{W}
- IC7 pad 7: A2 -> GND
- IC7 pad 8: A3 -> /IDE/~{RD}
- IC7 pad 9: RESET -> /IDE/~{WR}
- IC8 pad 1: IRQRS -> /Xosera_Bus/IRQRS
- IC8 pad 3: OIRQ -> /Xosera_Bus/OIRQ
- IC9 pad 1: A6 -> /Xosera_Bus/R~{W}
- IC9 pad 11: unconnected-(IC9-I10/~{OE}-Pad11) -> /Expansion_RAM/D7
- IC9 pad 12: unconnected-(IC9-IO8-Pad12) -> /Expansion_RAM/D6
- IC9 pad 13: A16 -> /Expansion_RAM/D5
- IC9 pad 14: A15 -> /Expansion_RAM/D4
- IC9 pad 15: A5 -> /Expansion_RAM/D3
- IC9 pad 16: UDS -> /Expansion_RAM/D2
- IC9 pad 17: LDS -> /Expansion_RAM/D1
- IC9 pad 18: IOSEL -> /Expansion_RAM/D0
- IC9 pad 19: SEL_1 -> /IDE/~{LSEL}
- IC9 pad 2: A7 -> BD0
- IC9 pad 20: +5V -> +5VD
- IC9 pad 3: A8 -> BD1
- IC9 pad 4: A9 -> BD2
- IC9 pad 5: unconnected-(IC9-I5-Pad5) -> BD3
- IC9 pad 6: unconnected-(IC9-I6-Pad6) -> BD4
- IC9 pad 7: unconnected-(IC9-I7-Pad7) -> BD5
- IC9 pad 8: unconnected-(IC9-I8-Pad8) -> BD6
- IC9 pad 9: unconnected-(IC9-I9-Pad9) -> BD7
- J1 pad 1: A1 -> /Xosera_Bus/A1
- J1 pad 11: A6 -> /Xosera_Bus/A6
- J1 pad 13: A7 -> /Xosera_Bus/A7
- J1 pad 14: unconnected-(J1-Pin_14-Pad14) -> /IDE/~{IRQ3}
- J1 pad 15: A8 -> /Xosera_Bus/A8
- J1 pad 16: IOSEL -> /Xosera_Bus/~{IOSEL}
- J1 pad 17: A9 -> /Xosera_Bus/A9
- J1 pad 18: unconnected-(J1-Pin_18-Pad18) -> /Xosera_Bus/~{EXPSEL}
- J1 pad 19: A10 -> /Xosera_Bus/A10
- J1 pad 20: FC0 -> /Xosera_Bus/FC0
- J1 pad 21: A11 -> /Xosera_Bus/A11
- J1 pad 22: FC1 -> /Xosera_Bus/FC1
- J1 pad 23: A12 -> /Xosera_Bus/A12
- J1 pad 24: FC2 -> /Xosera_Bus/FC2
- J1 pad 25: A13 -> /Xosera_Bus/A13
- J1 pad 26: unconnected-(J1-Pin_26-Pad26) -> /IDE/~{IRQ5}
- J1 pad 27: A14 -> /Xosera_Bus/A14
- J1 pad 29: A15 -> /Xosera_Bus/A15
- J1 pad 3: A2 -> /Xosera_Bus/A2
- J1 pad 30: unconnected-(J1-Pin_30-Pad30) -> /IDE/~{IRQ6}
- J1 pad 31: A16 -> /Xosera_Bus/A16
- J1 pad 32: LDS -> /Xosera_Bus/~{LDS}
- J1 pad 33: A17 -> /Xosera_Bus/A17
- J1 pad 34: UDS -> /Xosera_Bus/~{UDS}
- J1 pad 35: unconnected-(J1-Pin_35-Pad35) -> /Expansion_RAM/A18
- J1 pad 36: RESET -> /Xosera_Bus/~{RESET}
- J1 pad 37: unconnected-(J1-Pin_37-Pad37) -> /Expansion_RAM/A19
- J1 pad 38: 68_D15 -> /Xosera_Bus/5V_D15
- J1 pad 39: unconnected-(J1-Pin_39-Pad39) -> /Xosera_Bus/A20
- J1 pad 4: unconnected-(J1-Pin_4-Pad4) -> /Xosera_Bus/CLK
- J1 pad 40: 68_D14 -> /Xosera_Bus/5V_D14
- J1 pad 41: unconnected-(J1-Pin_41-Pad41) -> /Xosera_Bus/A21
- J1 pad 42: 68_D13 -> /Xosera_Bus/5V_D13
- J1 pad 43: unconnected-(J1-Pin_43-Pad43) -> /Xosera_Bus/A22
- J1 pad 44: 68_D12 -> /Xosera_Bus/5V_D12
- J1 pad 45: unconnected-(J1-Pin_45-Pad45) -> /Xosera_Bus/A23
- J1 pad 46: 68_D11 -> /Xosera_Bus/5V_D11
- J1 pad 47: AS -> /Xosera_Bus/~{AS}
- J1 pad 48: 68_D10 -> /Xosera_Bus/5V_D10
- J1 pad 5: A3 -> /Xosera_Bus/A3
- J1 pad 50: 68_D9 -> /Xosera_Bus/5V_D9
- J1 pad 52: 68_D8 -> /Xosera_Bus/5V_D8
- J1 pad 54: unconnected-(J1-Pin_54-Pad54) -> /Expansion_RAM/D7
- J1 pad 56: unconnected-(J1-Pin_56-Pad56) -> /Expansion_RAM/D6
- J1 pad 57: DTACK -> /Xosera_Bus/~{DTACK}
- J1 pad 58: unconnected-(J1-Pin_58-Pad58) -> /Expansion_RAM/D5
- J1 pad 59: RnW -> /Xosera_Bus/R~{W}
- J1 pad 60: unconnected-(J1-Pin_60-Pad60) -> /Expansion_RAM/D4
- J1 pad 61: unconnected-(J1-Pin_61-Pad61) -> /Expansion_RAM/D0
- J1 pad 62: unconnected-(J1-Pin_62-Pad62) -> /Expansion_RAM/D3
- J1 pad 63: unconnected-(J1-Pin_63-Pad63) -> /Expansion_RAM/D1
- J1 pad 64: unconnected-(J1-Pin_64-Pad64) -> /Expansion_RAM/D2
- J1 pad 7: A4 -> /Xosera_Bus/A4
- J1 pad 8: VPA -> /Xosera_Bus/~{VPA}
- J1 pad 9: A5 -> /Xosera_Bus/A5
- J10 pad 1: +3.3V -> +5V
- J10 pad 2: /Xosera_Bus/AUDIO_L -> /Xosera_Bus/AUDIO_R
- J10 pad 5: /Xosera_Bus/AUDIO_R -> /Xosera_Bus/AUDIO_L
- J10 pad 6: +5V -> +3.3V
- J3 pad 1: +3V3 -> GND
- J3 pad 3: GND -> +3V3
- J4 pad 1: +3V3 -> GND
- J4 pad 3: GND -> +3V3
- J5 pad 1: +3V3 -> GND
- J5 pad 3: GND -> +3V3
- J6 pad 1: /Xosera_HDMI/DKEN -> GND
- J6 pad 2: GND -> /Xosera_HDMI/DKEN
- JP1 pad 1: DTACK -> /Xosera_Bus/~{DTACK}
- JP1 pad 2: ODTACK -> /Xosera_Bus/~{ODTACK}
- JP2 pad 1: JBUS_RESET_N -> /Xosera_Bus/~{J3V3_RESET}
- L1 pad 1: +3V3 -> /Xosera_HDMI/VCC
- L1 pad 2: /Xosera_HDMI/VCC -> +3V3
- L2 pad 1: +3V3 -> /Xosera_HDMI/PVCC
- L2 pad 2: /Xosera_HDMI/PVCC -> +3V3
- L3 pad 1: +3V3 -> /Xosera_HDMI/TVDD
- L3 pad 2: /Xosera_HDMI/TVDD -> +3V3
- SJ8 pad 2: /Xosera_Bus/UD_IRQ -> /Xosera_Bus/XOSERA_IRQ
- TP19 pad 1: 68_D15 -> /Xosera_Bus/5V_D8
- TP19 pad 2: 68_D14 -> /Xosera_Bus/5V_D9
- TP19 pad 3: 68_D13 -> /Xosera_Bus/5V_D10
- TP19 pad 4: 68_D12 -> /Xosera_Bus/5V_D11
- TP19 pad 5: 68_D11 -> /Xosera_Bus/5V_D12
- TP19 pad 6: 68_D10 -> /Xosera_Bus/5V_D13
- TP19 pad 7: 68_D9 -> /Xosera_Bus/5V_D14
- TP19 pad 8: 68_D8 -> /Xosera_Bus/5V_D15
- TP20 pad 1: BUS_DATA7 -> /Xosera_Bus/3V3_D8
- TP20 pad 2: BUS_DATA6 -> /Xosera_Bus/3V3_D9
- TP20 pad 3: BUS_DATA5 -> /Xosera_Bus/3V3_D10
- TP20 pad 4: BUS_DATA4 -> /Xosera_Bus/3V3_D11
- TP20 pad 5: BUS_DATA3 -> /Xosera_Bus/3V3_D12
- TP20 pad 6: BUS_DATA2 -> /Xosera_Bus/3V3_D13
- TP20 pad 7: BUS_DATA1 -> /Xosera_Bus/3V3_D14
- TP20 pad 8: BUS_DATA0 -> /Xosera_Bus/3V3_D15
- TP21 pad 1: BUS_BYTESEL -> /Xosera_Bus/~{J3V3_RESET}
- TP21 pad 2: BUS_REG_NUM0 -> /Xosera_Bus/3V3_R~{W}
- TP21 pad 3: BUS_REG_NUM1 -> /Xosera_Bus/~{3V3_XOSERA_CS}
- TP21 pad 4: BUS_REG_NUM2 -> /Xosera_Bus/3V3_REG_NUM3
- TP21 pad 5: BUS_REG_NUM3 -> /Xosera_Bus/3V3_REG_NUM2
- TP21 pad 6: BUS_CS_N -> /Xosera_Bus/3V3_REG_NUM1
- TP21 pad 7: BUS_RD_NWR -> /Xosera_Bus/3V3_REG_NUM0
- TP21 pad 8: JBUS_RESET_N -> /Xosera_Bus/3V3_BYTESEL

Commit message: Fix Kicad weirdness
Parts:
- removed J9: 47589-0001, Connector_USB:USB_Micro-AB_Molex_47590-0001
- removed SJ2, SJ3: SHORT, Jumper:SolderJumper-2_P1.3mm_Bridged2Bar_RoundedPad1.0x1.5mm
- added J16: USB_C, Connector_USB:USB_C_Receptacle_Palconn_UTC16-G, F.Cu at (182.7, -15.6)
- added R34: 5.1K, Resistor_SMD:R_0805_2012Metric_Pad1.20x1.40mm_HandSolder, F.Cu at (174.5, -18.2)
- added R35: 5.1K, Resistor_SMD:R_0805_2012Metric_Pad1.20x1.40mm_HandSolder, F.Cu at (174.5, -15.3)
- added R36: 22R, Resistor_SMD:R_0805_2012Metric_Pad1.20x1.40mm_HandSolder, F.Cu at (174.5, -12.3)
- added R37: 22R, Resistor_SMD:R_0805_2012Metric_Pad1.20x1.40mm_HandSolder, F.Cu at (174.5, -9.39)
Connections:
- net /Xosera_Bus/AUDIO_L renamed /Audio_Filters/Audio_L_Filt
- net /Xosera_Bus/AUDIO_R renamed /Audio_Filters/Audio_R_Filt
- IC1 pad 1: Net-(IC1-CLK) -> Net-(IC1-DO)
- IC1 pad 3: Net-(IC1-CLK) -> /Xosera_FPGA/EE_DAT
- IC1 pad 4: Net-(IC1-CLK) -> /Xosera_FPGA/EE_CLK
- R4 pad 1: Net-(IC1-CLK) -> Net-(IC1-DO)
- R5 pad 2: Net-(IC1-CLK) -> Net-(IC1-DO)

Commit message: Initial layout, delete some useless things
Parts:
- removed C74: 10u, Capacitor_SMD:CP_Elec_6.3x5.4
- removed FID1, FID2, FID3, FID4, FID5, FID6: Fiducial, Fiducial:Fiducial_0.75mm_Mask1.5mm
- removed J14: Conn_02x07_Odd_Even, Connector_IDC:IDC-Header_2x07_P2.54mm_Vertical
- removed TP1, TP10, TP11, TP12, TP13, TP14, TP15, TP16, TP17, TP18, TP2, TP23, TP24, TP3, TP4, TP5, TP6, TP7, TP8, TP9: TestPoint, TestPoint:TestPoint_Pad_D1.0mm
- removed TP19, TP20, TP21: Conn_01x08_Male, Connector_PinHeader_2.54mm:PinHeader_1x08_P2.54mm_Vertical
- added C63: 100n, Capacitor_SMD:C_0402_1005Metric, F.Cu at (135.0, 100.6)
- added C64: 22pF, Capacitor_SMD:C_0603_1608Metric, F.Cu at (124.2, 113.4)
- added C65: 22pF, Capacitor_SMD:C_0603_1608Metric, F.Cu at (130.8, 113.4)
- added C66: 100n, Capacitor_SMD:C_0402_1005Metric, F.Cu at (129.0, 92.5)
- added IC15: ST16C2550IQ48TR-F, Package_QFP:TQFP-48_7x7mm_P0.5mm, F.Cu at (124.8, 97.1)
- added IC16: 74HC14, Package_SO:SOIC-14_3.9x8.7mm_P1.27mm, F.Cu at (136.7, 95.3)
- added J9: UART_A, Connector_PinHeader_2.54mm:PinHeader_1x06_P2.54mm_Vertical, F.Cu at (113.9, 92.4)
- added Q4: 2N3904, Package_TO_SOT_SMD:SOT-23, F.Cu at (97.7, 82.9)
- added R38: 500K, Resistor_SMD:R_0603_1608Metric, F.Cu at (127.5, 113.4)
- added R39: 150K, Resistor_SMD:R_0603_1608Metric, F.Cu at (101.2, 82.0)
- added SJ2: OPEN, Jumper:SolderJumper-2_P1.3mm_Open_RoundedPad1.0x1.5mm, F.Cu at (183.2, 48.9)
- added SJ3: SHORT, Jumper:SolderJumper-2_P1.3mm_Bridged_RoundedPad1.0x1.5mm, F.Cu at (181.4, 53.7)
- added U10: TPS22929D, Package_TO_SOT_SMD:SOT-23-6, F.Cu at (179.6, 48.9)
- added Y1: 3.6864MHz, Crystal:Crystal_SMD_HC49-SD, F.Cu at (127.5, 108.6)
- C13, C14, C17, C21, C26, C27, C31, C7, IC10, JP5, JP6, JP7, Q1, R13, SJ4, SJ5, SJ6, SJ7: moved to B.Cu
- IC7: value ATF1504AS-TQFP100 -> ATF1504AS-PLCC84; footprint Package_QFP:TQFP-100_14x14mm_P0.5mm -> Package_LCC:PLCC-84_THT-Socket
- J15: footprint Connector_IDC:IDC-Header_2x05_P2.54mm_Vertical -> Connector_PinHeader_2.54mm:PinHeader_2x05_P2.54mm_Vertical
- moved JP7 439.4 mm to (75.6, 99.9)
- moved JP6 439.4 mm to (75.6, 96.0)
- moved JP5 439.4 mm to (75.6, 91.9)
- moved TP22 435.6 mm to (75.7, 49.5)
- moved IC9 428.0 mm to (86.9, 107.6)
- moved C69 424.6 mm to (79.4, 113.8)
- moved C70 423.6 mm to (79.4, 98.4)
- moved IC13 416.7 mm to (86.9, 92.2)
- moved C72 415.6 mm to (87.8, 64.0), turned to 180 degrees
- moved IC14 414.7 mm to (103.5, 107.5)
- moved C62 411.7 mm to (190.2, 119.9)
- moved C68 411.4 mm to (91.9, 100.3)
- moved C67 410.9 mm to (91.9, 84.9)
- moved C75 409.9 mm to (110.5, 103.2), turned to -90 degrees
- moved C61 396.1 mm to (174.5, 119.9)
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Connections:
- net /Xosera_FPGA/USB_M renamed /Xosera_FPGA/USB_N
- C1 pad 1: +3.3V -> +3V3
- C11 pad 1: +3.3V -> +3V3
- C12 pad 1: +3.3V -> +3V3
- C13 pad 1: +3.3V -> +3V3
- C20 pad 1: +3.3V -> +3V3
- C22 pad 1: +3.3V -> +3V3
- C23 pad 1: +3.3V -> +3V3
- C24 pad 1: +3.3V -> +3V3
- C28 pad 1: +3.3V -> +3V3
- C30 pad 1: +3.3V -> +3V3
- C31 pad 1: +3.3V -> +3V3
- C48 pad 1: +3.3V -> +5V
- C49 pad 1: +3.3V -> +5V
- C5 pad 1: +5V -> Net-(IC3-VREGIN)
- C50 pad 1: +3.3V -> +3V3
- C51 pad 1: +3.3V -> +3V3
- C52 pad 1: +3.3V -> +3V3
- C53 pad 1: +3.3V -> +5V
- C54 pad 1: +3.3V -> +5V
- C56 pad 1: +5VD -> +5V
- C58 pad 1: +5VD -> +5V
- C59 pad 1: +3.3V -> +5V
- C60 pad 1: +3.3V -> +5V
- C61 pad 1: +3.3V -> +5V
- C62 pad 1: +3.3V -> +5V
- C67 pad 1: +5VD -> +5V
- C68 pad 1: +5VD -> +5V
- C69 pad 1: +5VD -> +5V
- C7 pad 1: +3.3V -> +3V3
- C70 pad 1: +5VD -> +5V
- C71 pad 1: +5VD -> +5V
- C72 pad 1: +5VD -> +5V
- C73 pad 1: +5VD -> +5V
- C75 pad 1: +5VD -> +5V
- D1 pad 2: +3.3V -> +3V3
- FB1 pad 1: +5V -> Net-(IC3-VREGIN)
- FB2 pad 2: +3.3V -> +3V3
- FB3 pad 2: +3.3V -> +3V3
- IC1 pad 6: +3.3V -> +3V3
- IC10 pad 8: +3.3V -> +3V3
- IC11 pad 16: +5VD -> +5V
- IC12 pad 16: +5VD -> +5V
- IC13 pad 20: +5VD -> +5V
- IC14 pad 20: +5VD -> +5V
- IC2 pad 22: +3.3V -> +3V3
- IC3 pad 12: +3.3V -> +3V3
- IC3 pad 16: Net-(IC3-ADBUS3) -> unconnected-(IC3-ADBUS3-Pad16)
- IC3 pad 18: Net-(IC3-ADBUS5) -> unconnected-(IC3-ADBUS5-Pad18)
- IC3 pad 21: Net-(IC3-ACBUS0) -> unconnected-(IC3-ACBUS0-Pad21)
- IC3 pad 24: +3.3V -> +3V3
- IC3 pad 25: Net-(IC3-ACBUS1) -> unconnected-(IC3-ACBUS1-Pad25)
- IC3 pad 26: Net-(IC3-ACBUS2) -> unconnected-(IC3-ACBUS2-Pad26)
- IC3 pad 27: Net-(IC3-ACBUS3) -> unconnected-(IC3-ACBUS3-Pad27)
- IC3 pad 28: Net-(IC3-ACBUS4) -> unconnected-(IC3-ACBUS4-Pad28)
- IC3 pad 29: Net-(IC3-ACBUS5) -> unconnected-(IC3-ACBUS5-Pad29)
- IC3 pad 30: Net-(IC3-ACBUS6) -> unconnected-(IC3-ACBUS6-Pad30)
- IC3 pad 31: Net-(IC3-ACBUS7) -> unconnected-(IC3-ACBUS7-Pad31)
- IC3 pad 32: Net-(IC3-ACBUS8) -> unconnected-(IC3-ACBUS8-Pad32)
- IC3 pad 33: Net-(IC3-ACBUS9) -> unconnected-(IC3-ACBUS9-Pad33)
- IC3 pad 34: +3.3V -> +3V3
- IC3 pad 40: +5V -> Net-(IC3-VREGIN)
- IC3 pad 46: +3.3V -> +3V3
- IC4 pad 5: +3.3V -> +3V3
- IC7 pad 4: /Xosera_Bus/~{IDE_CS} -> /UART/~{SEL}
- IC7 pad 41: /Xosera_Bus/RAM_EN_0 -> unconnected-(IC7-I/O-Pad41)
- IC9 pad 20: +5VD -> +5V
- J10 pad 6: +3.3V -> +3V3
- JP3 pad 1: +5VD -> +5V
- JP5 pad 1: Net-(IC13B-O0) -> Net-(IC13B-O2)
- JP5 pad 2: /IDE/~{IRQ3} -> /IDE/~{IRQ6}
- JP7 pad 1: Net-(IC13B-O2) -> Net-(IC13B-O0)
- JP7 pad 2: /IDE/~{IRQ6} -> /IDE/~{IRQ3}
- Q1 pad 4: +3.3V -> +3V3
- Q3 pad 1: +5VD -> +5V
- R1 pad 1: +3.3V -> +3V3
- R10 pad 2: +3.3V -> +3V3
- R11 pad 2: +3.3V -> +3V3
- R12 pad 2: +3.3V -> +3V3
- R28 pad 1: +5VD -> +5V
- R29 pad 1: +5VD -> +5V
- R3 pad 2: +3.3V -> +3V3
- R4 pad 2: +3.3V -> +3V3
- R7 pad 2: +3.3V -> +3V3
- R8 pad 2: +3.3V -> +3V3
- R9 pad 2: +3.3V -> +3V3
- SJ4 pad 1: +3.3V -> +3V3
- SJ6 pad 1: +3.3V -> +3V3
- TP22 pad 1: +5VD -> +5V
- U1 pad 8: +3.3V -> +3V3
- U2 pad 1: /Xosera_Bus/A5 -> /Xosera_Bus/A4
- U2 pad 10: /Expansion_RAM/D3 -> /Expansion_RAM/D0
- U2 pad 11: +3.3V -> +5V
- U2 pad 13: /Expansion_RAM/D4 -> /Expansion_RAM/D7
- U2 pad 14: /Expansion_RAM/D5 -> /Expansion_RAM/D6
- U2 pad 15: /Expansion_RAM/D6 -> /Expansion_RAM/D5
- U2 pad 16: /Expansion_RAM/D7 -> /Expansion_RAM/D4
- U2 pad 18: /Expansion_RAM/A19 -> /Xosera_Bus/A15
- U2 pad 19: /Expansion_RAM/A18 -> /Xosera_Bus/A16
- U2 pad 2: /Xosera_Bus/A4 -> /Xosera_Bus/A5
- U2 pad 21: /Xosera_Bus/A16 -> /Expansion_RAM/A18
- U2 pad 22: /Xosera_Bus/A15 -> /Expansion_RAM/A19
- U2 pad 33: +3.3V -> +5V
- U2 pad 7: /Expansion_RAM/D0 -> /Expansion_RAM/D3
- U2 pad 8: /Expansion_RAM/D1 -> /Expansion_RAM/D2
- U2 pad 9: /Expansion_RAM/D2 -> /Expansion_RAM/D1
- U3 pad 1: /Xosera_Bus/A5 -> /Xosera_Bus/A4
- U3 pad 10: /Expansion_RAM/D3 -> /Expansion_RAM/D0
- U3 pad 11: +3.3V -> +5V
- U3 pad 13: /Expansion_RAM/D4 -> /Expansion_RAM/D7
- U3 pad 14: /Expansion_RAM/D5 -> /Expansion_RAM/D6
- U3 pad 15: /Expansion_RAM/D6 -> /Expansion_RAM/D5
- U3 pad 16: /Expansion_RAM/D7 -> /Expansion_RAM/D4
- U3 pad 18: /Expansion_RAM/A19 -> /Xosera_Bus/A15
- U3 pad 19: /Expansion_RAM/A18 -> /Xosera_Bus/A16
- U3 pad 2: /Xosera_Bus/A4 -> /Xosera_Bus/A5
- U3 pad 21: /Xosera_Bus/A16 -> /Expansion_RAM/A18
- U3 pad 22: /Xosera_Bus/A15 -> /Expansion_RAM/A19
- U3 pad 33: +3.3V -> +5V
- U3 pad 7: /Expansion_RAM/D0 -> /Expansion_RAM/D3
- U3 pad 8: /Expansion_RAM/D1 -> /Expansion_RAM/D2
- U3 pad 9: /Expansion_RAM/D2 -> /Expansion_RAM/D1
- U4 pad 1: /Xosera_Bus/A5 -> /Xosera_Bus/A4
- U4 pad 10: /Expansion_RAM/D3 -> /Expansion_RAM/D0
- U4 pad 11: +3.3V -> +5V
- U4 pad 13: /Expansion_RAM/D4 -> /Expansion_RAM/D7
- U4 pad 14: /Expansion_RAM/D5 -> /Expansion_RAM/D6
- U4 pad 15: /Expansion_RAM/D6 -> /Expansion_RAM/D5
- U4 pad 16: /Expansion_RAM/D7 -> /Expansion_RAM/D4
- U4 pad 18: /Expansion_RAM/A19 -> /Xosera_Bus/A15
- U4 pad 19: /Expansion_RAM/A18 -> /Xosera_Bus/A16
- U4 pad 2: /Xosera_Bus/A4 -> /Xosera_Bus/A5
- U4 pad 21: /Xosera_Bus/A16 -> /Expansion_RAM/A18
- U4 pad 22: /Xosera_Bus/A15 -> /Expansion_RAM/A19
- U4 pad 33: +3.3V -> +5V
- U4 pad 7: /Expansion_RAM/D0 -> /Expansion_RAM/D3
- U4 pad 8: /Expansion_RAM/D1 -> /Expansion_RAM/D2
- U4 pad 9: /Expansion_RAM/D2 -> /Expansion_RAM/D1
- U5 pad 1: /Xosera_Bus/A5 -> /Xosera_Bus/A4
- U5 pad 10: /Expansion_RAM/D3 -> /Expansion_RAM/D0
- U5 pad 11: +3.3V -> +5V
- U5 pad 13: /Expansion_RAM/D4 -> /Expansion_RAM/D7
- U5 pad 14: /Expansion_RAM/D5 -> /Expansion_RAM/D6
- U5 pad 15: /Expansion_RAM/D6 -> /Expansion_RAM/D5
- U5 pad 16: /Expansion_RAM/D7 -> /Expansion_RAM/D4
- U5 pad 18: /Expansion_RAM/A19 -> /Xosera_Bus/A15
- U5 pad 19: /Expansion_RAM/A18 -> /Xosera_Bus/A16
- U5 pad 2: /Xosera_Bus/A4 -> /Xosera_Bus/A5
- U5 pad 21: /Xosera_Bus/A16 -> /Expansion_RAM/A18
- U5 pad 22: /Xosera_Bus/A15 -> /Expansion_RAM/A19
- U5 pad 33: +3.3V -> +5V
- U5 pad 7: /Expansion_RAM/D0 -> /Expansion_RAM/D3
- U5 pad 8: /Expansion_RAM/D1 -> /Expansion_RAM/D2
- U5 pad 9: /Expansion_RAM/D2 -> /Expansion_RAM/D1
- U6 pad 1: /Xosera_Bus/A5 -> /Xosera_Bus/A4
- U6 pad 10: /Expansion_RAM/D3 -> /Expansion_RAM/D0
- U6 pad 11: +3.3V -> +5V
- U6 pad 13: /Expansion_RAM/D4 -> /Expansion_RAM/D7
- U6 pad 14: /Expansion_RAM/D5 -> /Expansion_RAM/D6
- U6 pad 15: /Expansion_RAM/D6 -> /Expansion_RAM/D5
- U6 pad 16: /Expansion_RAM/D7 -> /Expansion_RAM/D4
- U6 pad 18: /Expansion_RAM/A19 -> /Xosera_Bus/A15
- U6 pad 19: /Expansion_RAM/A18 -> /Xosera_Bus/A16
- U6 pad 2: /Xosera_Bus/A4 -> /Xosera_Bus/A5
- U6 pad 21: /Xosera_Bus/A16 -> /Expansion_RAM/A18
- U6 pad 22: /Xosera_Bus/A15 -> /Expansion_RAM/A19
- U6 pad 33: +3.3V -> +5V
- U6 pad 7: /Expansion_RAM/D0 -> /Expansion_RAM/D3
- U6 pad 8: /Expansion_RAM/D1 -> /Expansion_RAM/D2
- U6 pad 9: /Expansion_RAM/D2 -> /Expansion_RAM/D1
- U7 pad 1: /Xosera_Bus/A5 -> /Xosera_Bus/A4
- U7 pad 10: /Expansion_RAM/D3 -> /Expansion_RAM/D0
- U7 pad 11: +3.3V -> +5V
- U7 pad 13: /Expansion_RAM/D4 -> /Expansion_RAM/D7
- U7 pad 14: /Expansion_RAM/D5 -> /Expansion_RAM/D6
- U7 pad 15: /Expansion_RAM/D6 -> /Expansion_RAM/D5
- U7 pad 16: /Expansion_RAM/D7 -> /Expansion_RAM/D4
- U7 pad 18: /Expansion_RAM/A19 -> /Xosera_Bus/A15
- U7 pad 19: /Expansion_RAM/A18 -> /Xosera_Bus/A16
- U7 pad 2: /Xosera_Bus/A4 -> /Xosera_Bus/A5
- U7 pad 21: /Xosera_Bus/A16 -> /Expansion_RAM/A18
- U7 pad 22: /Xosera_Bus/A15 -> /Expansion_RAM/A19
- U7 pad 33: +3.3V -> +5V
- U7 pad 7: /Expansion_RAM/D0 -> /Expansion_RAM/D3
- U7 pad 8: /Expansion_RAM/D1 -> /Expansion_RAM/D2
- U7 pad 9: /Expansion_RAM/D2 -> /Expansion_RAM/D1
- U8 pad 1: /Xosera_Bus/A5 -> /Xosera_Bus/A4
- U8 pad 10: /Expansion_RAM/D3 -> /Expansion_RAM/D0
- U8 pad 11: +3.3V -> +5V
- U8 pad 13: /Expansion_RAM/D4 -> /Expansion_RAM/D7
- U8 pad 14: /Expansion_RAM/D5 -> /Expansion_RAM/D6
- U8 pad 15: /Expansion_RAM/D6 -> /Expansion_RAM/D5
- U8 pad 16: /Expansion_RAM/D7 -> /Expansion_RAM/D4
- U8 pad 18: /Expansion_RAM/A19 -> /Xosera_Bus/A15
- U8 pad 19: /Expansion_RAM/A18 -> /Xosera_Bus/A16
- U8 pad 2: /Xosera_Bus/A4 -> /Xosera_Bus/A5
- U8 pad 21: /Xosera_Bus/A16 -> /Expansion_RAM/A18
- U8 pad 22: /Xosera_Bus/A15 -> /Expansion_RAM/A19
- U8 pad 33: +3.3V -> +5V
- U8 pad 7: /Expansion_RAM/D0 -> /Expansion_RAM/D3
- U8 pad 8: /Expansion_RAM/D1 -> /Expansion_RAM/D2
- U8 pad 9: /Expansion_RAM/D2 -> /Expansion_RAM/D1
- U9 pad 1: /Xosera_Bus/A5 -> /Xosera_Bus/A4
- U9 pad 10: /Expansion_RAM/D3 -> /Expansion_RAM/D0
- U9 pad 11: +3.3V -> +5V
- U9 pad 13: /Expansion_RAM/D4 -> /Expansion_RAM/D7
- U9 pad 14: /Expansion_RAM/D5 -> /Expansion_RAM/D6
- U9 pad 15: /Expansion_RAM/D6 -> /Expansion_RAM/D5
- U9 pad 16: /Expansion_RAM/D7 -> /Expansion_RAM/D4
- U9 pad 18: /Expansion_RAM/A19 -> /Xosera_Bus/A15
- U9 pad 19: /Expansion_RAM/A18 -> /Xosera_Bus/A16
- U9 pad 2: /Xosera_Bus/A4 -> /Xosera_Bus/A5
- U9 pad 21: /Xosera_Bus/A16 -> /Expansion_RAM/A18
- U9 pad 22: /Xosera_Bus/A15 -> /Expansion_RAM/A19
- U9 pad 33: +3.3V -> +5V
- U9 pad 7: /Expansion_RAM/D0 -> /Expansion_RAM/D3
- U9 pad 8: /Expansion_RAM/D1 -> /Expansion_RAM/D2
- U9 pad 9: /Expansion_RAM/D2 -> /Expansion_RAM/D1
Routing:
- net GND: track 0.00 -> 405.8 mm, vias 0 -> 96
- net +5V: track 0.00 -> 204.9 mm, vias 0 -> 59
- net +3V3: track 0.00 -> 112.3 mm, vias 0 -> 36
- net /Xosera_Bus/~{3V3_RESET}: track 0.00 -> 106.6 mm, vias 0 -> 2
- net /Xosera_FPGA/CDONE: track 0.00 -> 97.5 mm, vias 0 -> 2
- net /Xosera_HDMI/PVCC: track 0.00 -> 47.2 mm, vias 0 -> 2
- net /Xosera_HDMI/VCC: track 0.00 -> 43.8 mm, vias 0 -> 2
- net /Xosera_FPGA/V_USB: track 0.00 -> 41.4 mm, vias 0 -> 2
- net Net-(IC3-VREGIN): track 0.00 -> 37.7 mm, vias 0 -> 2
- net /Xosera_FPGA/FT_SCK: track 0.00 -> 31.0 mm, vias 0 -> 2
- net /Xosera_HDMI/TFADJ: track 0.00 -> 28.0 mm
- net /Xosera_Bus/XOSERA_IRQ: track 0.00 -> 27.2 mm, vias 0 -> 2
- net /Xosera_FPGA/EE_CS: track 0.00 -> 27.2 mm, vias 0 -> 2
- net /Xosera_HDMI/TVDD: track 0.00 -> 25.5 mm, vias 0 -> 2
- net /Xosera_FPGA/+1.2V_CORE: track 0.00 -> 25.1 mm, vias 0 -> 3
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- added copper zone on In2.Cu, net +3V3
- added copper zone on In2.Cu, net +5V
- added copper zone on In2.Cu, net /Xosera_FPGA/+1.2V_CORE
- added copper zone on In1.Cu, net GND
Other:
- outline, holes or cut-outs redrawn
- copper layers 2 -> 4
